Commit message: working version, with new gazebo

File: src/panda_description/description/models/panda/panda.urdf (robot description, URDF)
Before this commit: robot panda, 15 links, 14 joints
Joints:
- joint panda_finger_joint1: limit lower=-0.001 upper=0.04 effort=20. velocity=0.3 -> lower=-0.001 upper=0.04 effort=70. velocity=0.3
- joint panda_finger_joint2: limit lower=-0.001 upper=0.04 effort=20. velocity=0.3 -> lower=-0.001 upper=0.04 effort=70. velocity=0.3
